File: KiCad/ReCIA-AVR.sch (KiCad schematic (older format))
At the start: 18 parts, among them U1 AVR128DA64-I_MR, U2 74AHCT1G17, U3 TLC2932AIPWR, U5 8520_DIP

Commit message: Add net and resistor between PDF_OUT and VCO_IN for the AVR-version
Parts:
- added R3: 33, Resistor_SMD:R_0603_1608Metric_Pad0.98x0.95mm_HandSolder, symbol Device:R_Small
Connections:
- net labels added: PFD_OUT, VCO_IN, VCO_OUT
- net labels removed: EXT-CLK
- wire segments 67 -> 69
Changed lines of the file:
@@
 Text GLabel 9200 2350 1    50   Input ~ 0
 VCC
-Text GLabel 9900 3100 2    50   Input ~ 0
+Text GLabel 9550 3000 2    50   Input ~ 0
 GND
-Wire Wire Line
-	9550 3000 9900 3000
-Wire Wire Line
-	9900 3000 9900 3100
-Wire Wire Line
-	9550 3100 9900 3100
-Wire Wire Line
-	9550 3200 9900 3200
-Wire Wire Line
-	9900 3200 9900 3100
-Connection ~ 9900 3100
 Text Label 7700 2550 2    50   ~ 0
 LOGIC_VDD
@@
 Text GLabel 7850 3300 0    50   Input ~ 0
 GND
-Wire Wire Line
-	9550 3300 9900 3300
-Wire Wire Line
-	9900 3300 9900 3200
-Connection ~ 9900 3200
 Text GLabel 7850 3000 0    50   Input ~ 0
 E-CLK
@@
 	7650 2900 7850 2900
 Text Label 7650 2900 2    50   ~ 0
-EXT-CLK
+VCO_OUT
+$Comp
+L Device:R_Small R3
+U 1 1 678A30D6
+P 10000 3100
+F 0 "R3" V 10000 3100 50  0000 C CNN
+F 1 "33" V 9895 3100 50  0001 C CNN
+F 2 "Resistor_SMD:R_0603_1608Metric_Pad0.98x0.95mm_HandSolder" H 10000 3100 50  0001 C CNN
+F 3 "~" H 10000 3100 50  0001 C CNN
+	1    10000 3100
+	1    0    0    -1
+$EndComp
+Text Label 9550 2900 0    50   ~ 0
+VCO_IN
+Wire Wire Line
+	9550 3000 9550 3100
+Connection ~ 9550 3100
+Wire Wire Line
+	9550 3100 9550 3200
+Connection ~ 9550 3200
+Wire Wire Line
+	9550 3200 9550 3300
+Wire Wire Line
+	9550 2900 10000 2900
+Wire Wire Line
+	7850 3200 7600 3200
+Wire Wire Line
+	7600 3200 7600 3500
+Wire Wire Line
+	7600 3500 10000 3500
+Text Label 9550 3500 0    50   ~ 0
+PFD_OUT
+Wire Wire Line
+	10000 3500 10000 3200
+Wire Wire Line
+	10000 3000 10000 2900
 $EndSCHEMATC

Commit message: Add resistor and net for PLL FIN-B clk-count input signal from AVR pin 5 (PA7)
Parts:
- added R4: 33, Resistor_SMD:R_0603_1608Metric_Pad0.98x0.95mm_HandSolder, symbol Device:R_Small
Connections:
- net labels added: CLK_COUNT, FIN-B
- wire segments 69 -> 72
- no-connect marks 15 -> 14
Other:
- moved on the sheet: C6
Changed lines of the file:
@@
 Text GLabel 5150 5250 2    50   Input ~ 0
 GND
-Text GLabel 4000 3100 1    50   Input ~ 0
+Text GLabel 3750 3100 1    50   Input ~ 0
 VCC
-Text GLabel 4000 3300 3    50   Input ~ 0
+Text GLabel 3750 3300 3    50   Input ~ 0
 GND
 Text GLabel 5650 1250 2    50   Input ~ 0
@@
 Text GLabel 7000 3900 1    50   Input ~ 0
 GND
-NoConn ~ 5500 4850
 Text GLabel 4700 1650 1    50   Input ~ 0
 GND
@@
 L Device:C_Small C6
 U 1 1 66CAF364
-P 4000 3200
-F 0 "C6" H 4100 3200 50  0000 L CNN
-F 1 "0.01uF (0402)" V 3850 2950 50  0000 L CNN
-F 2 "Capacitor_SMD:C_0402_1005Metric" H 4000 3200 50  0001 C CNN
-F 3 "~" H 4000 3200 50  0001 C CNN
-	1    4000 3200
+P 3750 3200
+F 0 "C6" H 3850 3200 50  0000 L CNN
+F 1 "0.01uF (0402)" V 3600 2950 50  0000 L CNN
+F 2 "Capacitor_SMD:C_0402_1005Metric" H 3750 3200 50  0001 C CNN
+F 3 "~" H 3750 3200 50  0001 C CNN
+	1    3750 3200
 	1    0    0    -1
 $EndComp
-Wire Wire Line
-	4150 3250 4150 3300
-Wire Wire Line
-	4150 3300 4000 3300
-Wire Wire Line
-	4150 3250 4400 3250
-Wire Wire Line
-	4150 3150 4150 3100
-Wire Wire Line
-	4000 3100 4150 3100
-Wire Wire Line
-	4150 3150 4400 3150
 $Comp
 L Device:C_Small C2
@@
 Wire Wire Line
 	5150 5100 5150 5250
-NoConn ~ 4400 3050
 $Comp
 L ReCIA:74AHCT1G17 U2
@@
 Wire Wire Line
 	10000 3000 10000 2900
+$Comp
+L Device:R_Small R4
+U 1 1 678C2CF1
+P 7400 3300
+F 0 "R4" V 7296 3300 50  0000 C CNN
+F 1 "33" V 7295 3300 50  0001 C CNN
+F 2 "Resistor_SMD:R_0603_1608Metric_Pad0.98x0.95mm_HandSolder" H 7400 3300 50  0001 C CNN
+F 3 "~" H 7400 3300 50  0001 C CNN
+	1    7400 3300
+	0    1    1    0
+$EndComp
+Wire Wire Line
+	7850 3100 7500 3100
+Wire Wire Line
+	7500 3100 7500 3300
+Text Label 7500 3100 2    50   ~ 0
+FIN-B
+Text GLabel 7250 3300 0    50   Input ~ 0
+CLK_COUNT
+Wire Wire Line
+	7300 3300 7250 3300
+Text GLabel 4400 3050 0    50   Output ~ 0
+CLK_COUNT
+NoConn ~ 5500 4850
+Wire Wire Line
+	3750 3300 3850 3300
+Wire Wire Line
+	3850 3300 3850 3250
+Wire Wire Line
+	3850 3150 3850 3100
+Wire Wire Line
+	3850 3100 3750 3100
+Wire Wire Line
+	3850 3150 4400 3150
+Wire Wire Line
+	3850 3250 4400 3250
 $EndSCHEMATC

Commit message: Add pull-up resistor on SELECT-line and more placement and routing fixes
Parts:
- added R5: 33, Resistor_SMD:R_0603_1608Metric_Pad0.98x0.95mm_HandSolder, symbol Device:R_Small
Connections:
- net labels added: SELECT
- wire segments 72 -> 76
Other:
- moved on the sheet: R2
Changed lines of the file:
@@
 	7800 2150 7900 2150
 Wire Wire Line
-	7700 2350 7700 2700
+	7700 2350 7700 2600
 Wire Wire Line
 	7700 2700 7850 2700
@@
 Text GLabel 7850 3000 0    50   Input ~ 0
 E-CLK
-Text GLabel 7250 2750 0    50   Output ~ 0
+Text GLabel 7000 2750 0    50   Output ~ 0
 EXTCLK
 $Comp
 L Device:R_Small R2
 U 1 1 678932BF
-P 7400 2750
-F 0 "R2" V 7296 2750 50  0000 C CNN
-F 1 "33" V 7295 2750 50  0001 C CNN
-F 2 "Resistor_SMD:R_0603_1608Metric_Pad0.98x0.95mm_HandSolder" H 7400 2750 50  0001 C CNN
-F 3 "~" H 7400 2750 50  0001 C CNN
-	1    7400 2750
+P 7150 2750
+F 0 "R2" V 7046 2750 50  0000 C CNN
+F 1 "33" V 7045 2750 50  0001 C CNN
+F 2 "Resistor_SMD:R_0603_1608Metric_Pad0.98x0.95mm_HandSolder" H 7150 2750 50  0001 C CNN
+F 3 "~" H 7150 2750 50  0001 C CNN
+	1    7150 2750
 	0    1    1    0
 $EndComp
 Wire Wire Line
-	7300 2750 7250 2750
+	7050 2750 7000 2750
 Wire Wire Line
-	7650 2900 7650 2750
+	7400 2900 7400 2750
 Wire Wire Line
-	7650 2750 7500 2750
-Wire Wire Line
-	7650 2900 7850 2900
-Text Label 7650 2900 2    50   ~ 0
+	7400 2750 7250 2750
+Text Label 7400 2900 2    50   ~ 0
 VCO_OUT
 $Comp
@@
 Wire Wire Line
 	3850 3250 4400 3250
+$Comp
+L Device:R_Small R5
+U 1 1 6790992E
+P 7550 2800
+F 0 "R5" V 7446 2800 50  0000 C CNN
+F 1 "33" V 7445 2800 50  0001 C CNN
+F 2 "Resistor_SMD:R_0603_1608Metric_Pad0.98x0.95mm_HandSolder" H 7550 2800 50  0001 C CNN
+F 3 "~" H 7550 2800 50  0001 C CNN
+	1    7550 2800
+	0    1    1    0
+$EndComp
+Wire Wire Line
+	7400 2900 7850 2900
+Wire Wire Line
+	7450 2800 7450 2600
+Connection ~ 7700 2600
+Wire Wire Line
+	7700 2600 7700 2700
+Text Label 7650 2800 0    50   ~ 0
+SELECT
+Wire Wire Line
+	7650 2800 7850 2800
+Wire Wire Line
+	7450 2600 7700 2600
 $EndSCHEMATC

Commit message: Add 3.3k resistor and 0.22uF cap for the RBIAS-pin on the PLL
Parts:
- added C11: 0.22uF, Capacitor_SMD:C_0603_1608Metric_Pad1.08x0.95mm_HandSolder, symbol Device:C_Small
- added R6: 3k3, Resistor_SMD:R_0603_1608Metric_Pad0.98x0.95mm_HandSolder, symbol Device:R_Small
- renumbered C2 to C10, C10 to C2, C8 to C3, C3 to C8
Connections:
- net labels added: RBIAS
- wire segments 76 -> 81
Changed lines of the file:
@@
 $EndComp
 $Comp
-L Device:C_Small C2
+L Device:C_Small C10
 U 1 1 66CBB25E
 P 5050 5250
-F 0 "C2" V 4950 5300 50  0000 L CNN
+F 0 "C10" V 4950 5300 50  0000 L CNN
 F 1 "0.1uF (0603)" V 4850 4900 50  0000 L CNN
 F 2 "Capacitor_SMD:C_0603_1608Metric_Pad1.08x0.95mm_HandSolder" H 5050 5250 50  0001 C CNN
@@
 	6850 4100 7000 4100
 $Comp
-L Device:C_Small C3
+L Device:C_Small C8
 U 1 1 66CC3875
 P 7000 4000
-F 0 "C3" H 6800 3950 50  0000 L CNN
+F 0 "C8" H 6800 3950 50  0000 L CNN
 F 1 "0.1uF (0603)" H 6400 4050 50  0000 L CNN
 F 2 "Capacitor_SMD:C_0603_1608Metric_Pad1.08x0.95mm_HandSolder" H 7000 4000 50  0001 C CNN
@@
 	9550 2700 9700 2700
 $Comp
-L Device:C_Small C8
+L Device:C_Small C3
 U 1 1 67831839
 P 7900 2250
-F 0 "C8" H 7800 2250 50  0000 R CNN
+F 0 "C3" H 7800 2250 50  0000 R CNN
 F 1 "10uF" H 7800 2150 50  0000 R CNN
 F 2 "Capacitor_SMD:C_0805_2012Metric_Pad1.18x1.45mm_HandSolder" H 7900 2250 50  0001 C CNN
@@
 $EndComp
 $Comp
-L Device:C_Small C10
+L Device:C_Small C2
 U 1 1 67833368
 P 10250 2600
-F 0 "C10" H 10050 2600 50  0000 L CNN
+F 0 "C2" H 10000 2600 50  0000 L CNN
 F 1 "10uF" H 10000 2500 50  0000 L CNN
 F 2 "Capacitor_SMD:C_0805_2012Metric_Pad1.18x1.45mm_HandSolder" H 10250 2600 50  0001 C CNN
@@
 Text Label 7700 2550 2    50   ~ 0
 LOGIC_VDD
-Text Label 10550 2700 0    50   ~ 0
+Text Label 10750 2700 0    50   ~ 0
 VCO_VDD
-Wire Wire Line
-	10550 2700 10250 2700
 Connection ~ 10250 2700
 Text GLabel 7850 3300 0    50   Input ~ 0
@@
 Wire Wire Line
 	7450 2600 7700 2600
+$Comp
+L Device:C_Small C11
+U 1 1 67941D76
+P 10200 2900
+F 0 "C11" H 10150 3000 50  0000 R CNN
+F 1 "0.22uF" H 10150 3100 50  0000 R CNN
+F 2 "Capacitor_SMD:C_0603_1608Metric_Pad1.08x0.95mm_HandSolder" H 10200 2900 50  0001 C CNN
+F 3 "~" H 10200 2900 50  0001 C CNN
+	1    10200 2900
+	-1   0    0    1
+$EndComp
+Text GLabel 10200 3000 3    50   Input ~ 0
+GND
+Wire Wire Line
+	10200 2800 9550 2800
+$Comp
+L Device:R_Small R6
+U 1 1 67945075
+P 10450 2800
+F 0 "R6" V 10450 2800 50  0000 C CNN
+F 1 "3k3" V 10345 2800 50  0001 C CNN
+F 2 "Resistor_SMD:R_0603_1608Metric_Pad0.98x0.95mm_HandSolder" H 10450 2800 50  0001 C CNN
+F 3 "~" H 10450 2800 50  0001 C CNN
+	1    10450 2800
+	0    1    1    0
+$EndComp
+Wire Wire Line
+	10200 2800 10350 2800
+Connection ~ 10200 2800
+Wire Wire Line
+	10250 2700 10600 2700
+Wire Wire Line
+	10550 2800 10600 2800
+Wire Wire Line
+	10600 2800 10600 2700
+Connection ~ 10600 2700
+Wire Wire Line
+	10600 2700 10750 2700
+Text Label 9550 2800 0    50   ~ 0
+RBIAS
 $EndSCHEMATC

Commit message: Add cap for the VCO_IN-pin on the PLL
Parts:
- added C6: 0.1uF, Capacitor_SMD:C_0603_1608Metric_Pad1.08x0.95mm_HandSolder, symbol Device:C_Small
- renumbered C6 to C12
Connections:
- wire segments 81 -> 84
Other:
- moved on the sheet: C11, R6
Changed lines of the file:
@@
 NoConn ~ 6300 1650
 $Comp
-L Device:C_Small C6
+L Device:C_Small C12
 U 1 1 66CAF364
 P 3750 3200
-F 0 "C6" H 3850 3200 50  0000 L CNN
+F 0 "C12" H 3850 3200 50  0000 L CNN
 F 1 "0.01uF (0402)" V 3600 2950 50  0000 L CNN
 F 2 "Capacitor_SMD:C_0402_1005Metric" H 3750 3200 50  0001 C CNN
@@
 	9550 3200 9550 3300
 Wire Wire Line
-	9550 2900 10000 2900
+	9550 2900 9850 2900
 Wire Wire Line
 	7850 3200 7600 3200
@@
 L Device:C_Small C11
 U 1 1 67941D76
-P 10200 2900
-F 0 "C11" H 10150 3000 50  0000 R CNN
-F 1 "0.22uF" H 10150 3100 50  0000 R CNN
-F 2 "Capacitor_SMD:C_0603_1608Metric_Pad1.08x0.95mm_HandSolder" H 10200 2900 50  0001 C CNN
-F 3 "~" H 10200 2900 50  0001 C CNN
-	1    10200 2900
-	-1   0    0    1
-$EndComp
-Text GLabel 10200 3000 3    50   Input ~ 0
-GND
-Wire Wire Line
-	10200 2800 9550 2800
+P 10500 2900
+F 0 "C11" H 10450 3000 50  0000 R CNN
+F 1 "0.22uF" H 10450 3100 50  0000 R CNN
+F 2 "Capacitor_SMD:C_0603_1608Metric_Pad1.08x0.95mm_HandSolder" H 10500 2900 50  0001 C CNN
+F 3 "~" H 10500 2900 50  0001 C CNN
+	1    10500 2900
+	-1   0    0    1
+$EndComp
+Text GLabel 10500 3000 3    50   Input ~ 0
+GND
 $Comp
 L Device:R_Small R6
 U 1 1 67945075
-P 10450 2800
-F 0 "R6" V 10450 2800 50  0000 C CNN
-F 1 "3k3" V 10345 2800 50  0001 C CNN
-F 2 "Resistor_SMD:R_0603_1608Metric_Pad0.98x0.95mm_HandSolder" H 10450 2800 50  0001 C CNN
-F 3 "~" H 10450 2800 50  0001 C CNN
-	1    10450 2800
+P 10750 2800
+F 0 "R6" V 10750 2800 50  0000 C CNN
+F 1 "3k3" V 10645 2800 50  0001 C CNN
+F 2 "Resistor_SMD:R_0603_1608Metric_Pad0.98x0.95mm_HandSolder" H 10750 2800 50  0001 C CNN
+F 3 "~" H 10750 2800 50  0001 C CNN
+	1    10750 2800
 	0    1    1    0
 $EndComp
 Wire Wire Line
-	10200 2800 10350 2800
-Connection ~ 10200 2800
-Wire Wire Line
-	10250 2700 10600 2700
-Wire Wire Line
-	10550 2800 10600 2800
-Wire Wire Line
-	10600 2800 10600 2700
-Connection ~ 10600 2700
-Wire Wire Line
-	10600 2700 10750 2700
+	10500 2800 10650 2800
+Connection ~ 10500 2800
+Wire Wire Line
+	10850 2800 10900 2800
+Wire Wire Line
+	10900 2800 10900 2700
 Text Label 9550 2800 0    50   ~ 0
 RBIAS
+$Comp
+L Device:C_Small C6
+U 1 1 6796867A
+P 9850 3100
+F 0 "C6" H 9900 3200 50  0000 L CNN
+F 1 "0.1uF" H 9250 3150 50  0001 L CNN
+F 2 "Capacitor_SMD:C_0603_1608Metric_Pad1.08x0.95mm_HandSolder" H 9850 3100 50  0001 C CNN
+F 3 "~" H 9850 3100 50  0001 C CNN
+	1    9850 3100
+	-1   0    0    1
+$EndComp
+Wire Wire Line
+	9850 3200 9850 3300
+Wire Wire Line
+	9850 3300 9550 3300
+Connection ~ 9550 3300
+Wire Wire Line
+	9850 3000 9850 2900
+Connection ~ 9850 2900
+Wire Wire Line
+	9850 2900 10000 2900
+Wire Wire Line
+	10250 2700 10900 2700
+Wire Wire Line
+	9550 2800 10500 2800
 $EndSCHEMATC

Commit message: Change from 0805 to 1206 size on C2 and C3
Parts:
- C2, C3: footprint Capacitor_SMD:C_0805_2012Metric_Pad1.18x1.45mm_HandSolder -> Capacitor_SMD:C_1206_3216Metric_Pad1.33x1.80mm_HandSolder
- renumbered C8 to C11, C11 to C8
Other:
- moved on the sheet: C2, C3, C6, C7, C8, C9, R2, R3, R4, R5, R6

Commit message: Add resistor and cap on VCO_IN line
Parts:
- added C13: 0.1uF, Capacitor_SMD:C_0603_1608Metric_Pad1.08x0.95mm_HandSolder, symbol Device:C_Small
- added R7: 33, Resistor_SMD:R_0603_1608Metric_Pad0.98x0.95mm_HandSolder, symbol Device:R_Small
Connections:
- wire segments 84 -> 89
Changed lines of the file:
@@
 Text Label 7650 1400 2    50   ~ 0
 LOGIC_VDD
-Text Label 10700 1550 0    50   ~ 0
+Text Label 10500 1550 0    50   ~ 0
 VCO_VDD
 Connection ~ 10200 1550
@@
 U 1 1 678A30D6
 P 9950 1950
-F 0 "R3" V 9950 1950 50  0000 C CNN
+F 0 "R3" H 10050 1950 50  0000 C CNN
 F 1 "33" V 9845 1950 50  0001 C CNN
 F 2 "Resistor_SMD:R_0603_1608Metric_Pad0.98x0.95mm_HandSolder" H 9950 1950 50  0001 C CNN
@@
 Wire Wire Line
 	9500 1650 10450 1650
+$Comp
+L Device:R_Small R7
+U 1 1 679B48E0
+P 10150 1750
+F 0 "R7" V 10250 1750 50  0000 C CNN
+F 1 "33" V 10045 1750 50  0001 C CNN
+F 2 "Resistor_SMD:R_0603_1608Metric_Pad0.98x0.95mm_HandSolder" H 10150 1750 50  0001 C CNN
+F 3 "~" H 10150 1750 50  0001 C CNN
+	1    10150 1750
+	0    1    1    0
+$EndComp
+Wire Wire Line
+	9950 1750 10050 1750
+Connection ~ 9950 1750
+Wire Wire Line
+	10250 1750 10350 1750
+Wire Wire Line
+	10350 1750 10350 2150
+$Comp
+L Device:C_Small C13
+U 1 1 679B97A4
+P 10150 2150
+F 0 "C13" V 10250 2100 50  0000 L CNN
+F 1 "0.1uF" H 9550 2200 50  0001 L CNN
+F 2 "Capacitor_SMD:C_0603_1608Metric_Pad1.08x0.95mm_HandSolder" H 10150 2150 50  0001 C CNN
+F 3 "~" H 10150 2150 50  0001 C CNN
+	1    10150 2150
+	0    -1   -1   0
+$EndComp
+Wire Wire Line
+	10050 2150 9800 2150
+Connection ~ 9800 2150
+Wire Wire Line
+	10250 2150 10350 2150
 $EndSCHEMATC

Commit message: Fixed caps and resistor references enumeration, more routing and small fixes positioning vias
Parts:
- R7: renamed from R5; value 33 -> 10k
- renumbered C8 to C7, C9 to C8, C7 to C9, R6 to R1, R3 to R2, R7 to R3, R2 to R4, R4 to R5, R1 to R6
Changed lines of the file:
@@
 	2200 2100 2200 1900
 $Comp
-L Device:R_Small R1
+L Device:R_Small R6
 U 1 1 677C3D65
 P 3600 1600
-F 0 "R1" V 3496 1600 50  0000 C CNN
+F 0 "R6" V 3496 1600 50  0000 C CNN
 F 1 "33" V 3495 1600 50  0001 C CNN
 F 2 "Resistor_SMD:R_0603_1608Metric_Pad0.98x0.95mm_HandSolder" H 3600 1600 50  0001 C CNN
@@
 	9650 1450 9650 1550
 $Comp
-L Device:C_Small C7
+L Device:C_Small C9
 U 1 1 67838FC9
 P 7650 1100
-F 0 "C7" H 7750 1100 50  0000 L CNN
+F 0 "C9" H 7750 1100 50  0000 L CNN
 F 1 "0.01uF" H 7750 1000 50  0000 L CNN
 F 2 "Capacitor_SMD:C_0603_1608Metric_Pad1.08x0.95mm_HandSolder" H 7650 1100 50  0001 C CNN
@@
 Connection ~ 7850 1200
 $Comp
-L Device:C_Small C9
+L Device:C_Small C8
 U 1 1 6783A777
 P 10000 1450
-F 0 "C9" H 10100 1450 50  0000 L CNN
+F 0 "C8" H 10100 1450 50  0000 L CNN
 F 1 "0.01uF" H 10000 1350 50  0000 L CNN
 F 2 "Capacitor_SMD:C_0603_1608Metric_Pad1.08x0.95mm_HandSolder" H 10000 1450 50  0001 C CNN
@@
 EXTCLK
 $Comp
-L Device:R_Small R2
+L Device:R_Small R4
 U 1 1 678932BF
 P 7100 1600
-F 0 "R2" V 6996 1600 50  0000 C CNN
+F 0 "R4" V 6996 1600 50  0000 C CNN
 F 1 "33" V 6995 1600 50  0001 C CNN
 F 2 "Resistor_SMD:R_0603_1608Metric_Pad0.98x0.95mm_HandSolder" H 7100 1600 50  0001 C CNN
@@
 VCO_OUT
 $Comp
-L Device:R_Small R3
+L Device:R_Small R2
 U 1 1 678A30D6
 P 9950 1950
-F 0 "R3" H 10050 1950 50  0000 C CNN
+F 0 "R2" H 10050 1950 50  0000 C CNN
 F 1 "33" V 9845 1950 50  0001 C CNN
 F 2 "Resistor_SMD:R_0603_1608Metric_Pad0.98x0.95mm_HandSolder" H 9950 1950 50  0001 C CNN
@@
 	9950 1850 9950 1750
 $Comp
-L Device:R_Small R4
+L Device:R_Small R5
 U 1 1 678C2CF1
 P 7350 2150
-F 0 "R4" V 7246 2150 50  0000 C CNN
+F 0 "R5" V 7246 2150 50  0000 C CNN
 F 1 "33" V 7245 2150 50  0001 C CNN
 F 2 "Resistor_SMD:R_0603_1608Metric_Pad0.98x0.95mm_HandSolder" H 7350 2150 50  0001 C CNN
@@
 	3850 3250 4400 3250
 $Comp
-L Device:R_Small R5
+L Device:R_Small R7
 U 1 1 6790992E
 P 7500 1650
-F 0 "R5" V 7396 1650 50  0000 C CNN
-F 1 "33" V 7395 1650 50  0001 C CNN
+F 0 "R7" V 7396 1650 50  0000 C CNN
+F 1 "10k" V 7395 1650 50  0001 C CNN
 F 2 "Resistor_SMD:R_0603_1608Metric_Pad0.98x0.95mm_HandSolder" H 7500 1650 50  0001 C CNN
 F 3 "~" H 7500 1650 50  0001 C CNN
@@
 	7400 1450 7650 1450
 $Comp
-L Device:C_Small C8
+L Device:C_Small C7
 U 1 1 67941D76
 P 10450 1750
-F 0 "C8" H 10400 1850 50  0000 R CNN
+F 0 "C7" H 10400 1850 50  0000 R CNN
 F 1 "0.22uF" H 10400 1950 50  0000 R CNN
 F 2 "Capacitor_SMD:C_0603_1608Metric_Pad1.08x0.95mm_HandSolder" H 10450 1750 50  0001 C CNN
@@
 Text GLabel 10450 1850 3    50   Input ~ 0
 GND
-$Comp
-L Device:R_Small R6
-U 1 1 67945075
-P 10700 1650
-F 0 "R6" V 10700 1650 50  0000 C CNN
-F 1 "3k3" V 10595 1650 50  0001 C CNN
-F 2 "Resistor_SMD:R_0603_1608Metric_Pad0.98x0.95mm_HandSolder" H 10700 1650 50  0001 C CNN
-F 3 "~" H 10700 1650 50  0001 C CNN
-	1    10700 1650
-	0    1    1    0
-$EndComp
 Wire Wire Line
 	10450 1650 10600 1650
@@
 Wire Wire Line
 	9500 1650 10450 1650
-$Comp
-L Device:R_Small R7
-U 1 1 679B48E0
-P 10150 1750
-F 0 "R7" V 10250 1750 50  0000 C CNN
-F 1 "33" V 10045 1750 50  0001 C CNN
-F 2 "Resistor_SMD:R_0603_1608Metric_Pad0.98x0.95mm_HandSolder" H 10150 1750 50  0001 C CNN
-F 3 "~" H 10150 1750 50  0001 C CNN
-	1    10150 1750
-	0    1    1    0
-$EndComp
 Wire Wire Line
 	9950 1750 10050 1750
@@
 Wire Wire Line
 	10250 2150 10350 2150
+$Comp
+L Device:R_Small R1
+U 1 1 67945075
+P 10700 1650
+F 0 "R1" V 10800 1650 50  0000 C CNN
+F 1 "3k3" V 10595 1650 50  0001 C CNN
+F 2 "Resistor_SMD:R_0603_1608Metric_Pad0.98x0.95mm_HandSolder" H 10700 1650 50  0001 C CNN
+F 3 "~" H 10700 1650 50  0001 C CNN
+	1    10700 1650
+	0    1    1    0
+$EndComp
+$Comp
+L Device:R_Small R3
+U 1 1 679B48E0
+P 10150 1750
+F 0 "R3" V 10250 1750 50  0000 C CNN
+F 1 "33" V 10045 1750 50  0001 C CNN
+F 2 "Resistor_SMD:R_0603_1608Metric_Pad0.98x0.95mm_HandSolder" H 10150 1750 50  0001 C CNN
+F 3 "~" H 10150 1750 50  0001 C CNN
+	1    10150 1750
+	0    1    1    0
+$EndComp
 $EndSCHEMATC
